File: Hardware/Qwiic RFID - IDXXLA.brd (EAGLE design)
At the start: 25.4 x 30.5 mm, 60 parts, among them J2 SMD, J3 PTH, J4 SMD, J8 AVR_SPI_PROG_3X2TESTPOINTS, Q1 600mA/40V, U1 ATTINY84-ARDUINO, U2 ID-12/20SMD

Commit message: Firmware almost finalized, I2C data lines and UART lines fixed on board
Parts:
- moved U$2 0.38 mm to (14.1, 9.91)
Connections:
- removed net SCL: J2.4, J3.4, J4.4
- removed net SDA: J2.3, J3.3, J4.3
- net DATA_UART: now also U1.11; no longer U1.3
- net SCL/SCK: now also J2.4, J3.4, J4.4
- net SDA/MOSI: now also J2.3, J3.3, J4.3
Routing:
- net SCL/SCK: track 10.5 -> 57.4 mm, vias 0 -> 3
- net SDA/MOSI: track 5.67 -> 51.0 mm, vias 0 -> 3
- net SDA: track 42.4 -> 0.00 mm, vias 1 -> 0
- net SCL: track 42.2 -> 0.00 mm, vias 1 -> 0
- net DATA_UART: track 10.1 -> 17.1 mm
- net GND: vias 17 -> 18
