File: Hardware/Qwiic RFID - IDXXLA.sch (EAGLE design)
At the start: 35 parts, among them J2 SMD, J3 PTH, J4 SMD, J8 AVR_SPI_PROG_3X2TESTPOINTS, Q1 600mA/40V, U1 ATTINY84-ARDUINO, U2 ID-12/20SMD

Commit message: Panel for x02
Other:
- note added: "X02"
- note removed: "X01"
Changed lines of the file:
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@@
 <sheet>
 <plain>
-<text x="237.744" y="7.366" size="2.54" layer="94" font="vector">X01</text>
+<text x="237.744" y="7.366" size="2.54" layer="94" font="vector">X02</text>
 <wire x1="0" y1="83.82" x2="81.28" y2="83.82" width="0.2032" layer="97" style="shortdash"/>
 <text x="86.36" y="76.2" size="2.54" layer="94" font="vector">Buzzer and Power LED</text>

Commit message: Cleanup and ReadMe
Parts:
- J2, J4: value SMD -> (none); device SparkX:I2C_STANDARDJS-1MM -> SparkFun-Connectors:QWIIC_CONNECTORJS-1MM
Connections:
- net 3.3V: now also J2.2, J4.2; no longer J2.VCC, J4.VCC
- net GND: now also J2.1, J4.1; no longer J2.GND, J4.GND
- net SCL/SCK: now also J2.4, J4.4; no longer J2.SCL, J4.SCL
- net SDA/MOSI: now also J2.3, J4.3; no longer J2.SDA, J4.SDA
Changed lines of the file:
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@@
 <part name="SUPPLY1" library="SparkFun-PowerSymbols" deviceset="3.3V" device=""/>
 <part name="SUPPLY4" library="SparkFun-PowerSymbols" deviceset="3.3V" device=""/>
-<part name="J2" library="SparkX" deviceset="I2C_STANDARD" device="JS-1MM" value="SMD"/>
+<part name="J2" library="SparkFun-Connectors" deviceset="QWIIC_CONNECTOR" device="JS-1MM"/>
 <part name="GND6" library="SparkFun" deviceset="GND" device=""/>
 <part name="SUPPLY7" library="SparkFun-PowerSymbols" deviceset="3.3V" device=""/>
@@
 <part name="FRAME1" library="SparkFun-Aesthetics" deviceset="FRAME-LETTER" device=""/>
 <part name="SUPPLY8" library="SparkFun-PowerSymbols" deviceset="3.3V" device=""/>
-<part name="J4" library="SparkX" deviceset="I2C_STANDARD" device="JS-1MM" value="SMD"/>
+<part name="J4" library="SparkFun-Connectors" deviceset="QWIIC_CONNECTOR" device="JS-1MM"/>
 <part name="GND8" library="SparkFun" deviceset="GND" device=""/>
 <part name="LOGO1" library="SparkFun-Aesthetics" deviceset="OSHW-LOGO" device="MINI"/>
@@
 </segment>
 <segment>
-<pinref part="J2" gate="G$1" pin="VCC"/>
+<pinref part="J2" gate="G$1" pin="2"/>
 <wire x1="27.94" y1="48.26" x2="25.4" y2="48.26" width="0.1524" layer="91"/>
 <wire x1="25.4" y1="48.26" x2="25.4" y2="55.88" width="0.1524" layer="91"/>
@@
 </segment>
 <segment>
-<pinref part="J4" gate="G$1" pin="VCC"/>
+<pinref part="J4" gate="G$1" pin="2"/>
 <wire x1="27.94" y1="20.32" x2="25.4" y2="20.32" width="0.1524" layer="91"/>
 <wire x1="25.4" y1="20.32" x2="25.4" y2="27.94" width="0.1524" layer="91"/>
@@
 <net name="GND" class="0">
 <segment>
-<pinref part="J2" gate="G$1" pin="GND"/>
+<pinref part="J2" gate="G$1" pin="1"/>
 <wire x1="27.94" y1="45.72" x2="25.4" y2="45.72" width="0.1524" layer="91"/>
 <wire x1="25.4" y1="45.72" x2="25.4" y2="43.18" width="0.1524" layer="91"/>
@@
 </segment>
 <segment>
-<pinref part="J4" gate="G$1" pin="GND"/>
+<pinref part="J4" gate="G$1" pin="1"/>
 <wire x1="27.94" y1="17.78" x2="25.4" y2="17.78" width="0.1524" layer="91"/>
 <wire x1="25.4" y1="17.78" x2="25.4" y2="15.24" width="0.1524" layer="91"/>
@@
 </segment>
 <segment>
-<pinref part="J2" gate="G$1" pin="SCL"/>
+<pinref part="J2" gate="G$1" pin="4"/>
 <wire x1="27.94" y1="53.34" x2="22.86" y2="53.34" width="0.1524" layer="91"/>
 <label x="22.86" y="53.34" size="1.27" layer="95" font="vector" rot="R180" xref="yes"/>
@@
 </segment>
 <segment>
-<pinref part="J4" gate="G$1" pin="SCL"/>
+<pinref part="J4" gate="G$1" pin="4"/>
 <wire x1="27.94" y1="25.4" x2="22.86" y2="25.4" width="0.1524" layer="91"/>
 <label x="22.86" y="25.4" size="1.27" layer="95" font="vector" rot="R180" xref="yes"/>
@@
 </segment>
 <segment>
-<pinref part="J2" gate="G$1" pin="SDA"/>
+<pinref part="J2" gate="G$1" pin="3"/>
 <wire x1="27.94" y1="50.8" x2="22.86" y2="50.8" width="0.1524" layer="91"/>
 <label x="22.86" y="50.8" size="1.27" layer="95" font="vector" rot="R180" xref="yes"/>
@@
 </segment>
 <segment>
-<pinref part="J4" gate="G$1" pin="SDA"/>
+<pinref part="J4" gate="G$1" pin="3"/>
 <wire x1="27.94" y1="22.86" x2="22.86" y2="22.86" width="0.1524" layer="91"/>
 <label x="22.86" y="22.86" size="1.27" layer="95" font="vector" rot="R180" xref="yes"/>
